File: sofaboard/sofaboard.kicad_pcb (KiCad board)
At the start: 2 copper layers, 301 x 111.8 mm, 179 parts, among them J1 USB_B_Micro, SW1 SW_Push, SW10 SW_Push, SW11 SW_Push, SW12 SW_Push, SW13 SW_Push, SW14 SW_Push, SW15 SW_Push, SW16 SW_Push, SW17 SW_Push, SW18 SW_Push, SW19 SW_Push, SW2 SW_Push, SW20 SW_Push, SW21 SW_Push, SW22 SW_Push, SW23 SW_Push, SW24 SW_Push, SW25 SW_Push, SW26 SW_Push, SW27 SW_Push, SW28 SW_Push, SW29 SW_Push, SW3 SW_Push, SW30 SW_Push, SW31 SW_Push, SW32 SW_Push, SW33 SW_Push, SW34 SW_Push, SW35 SW_Push, SW36 SW_Push, SW37 SW_Push, SW38 SW_Push, SW39 SW_Push, SW4 SW_Push, SW40 SW_Push, SW41 SW_Push, SW42 SW_Push, SW43 SW_Push, SW44 SW_Push, SW45 SW_Push, SW46 SW_Push, SW47 SW_Push, SW48 SW_Push, SW49 SW_Push, SW5 SW_Push, SW50 SW_Push, SW51 SW_Push, SW52 SW_Push, SW53 SW_Push, SW54 SW_Push, SW55 SW_Push, SW56 SW_Push, SW57 SW_Push, SW58 SW_Push, SW59 SW_Push, SW6 SW_Push, SW60 SW_Push, SW61 SW_Push, SW62 SW_Push, SW63 SW_Push, SW64 SW_Push, SW65 SW_Push, SW66 SW_Push, SW67 SW_Push, SW68 SW_Push, SW69 SW_Push, SW7 SW_Push, SW70 SW_Push, SW71 SW_Push, SW72 SW_Push, SW73 SW_Push, SW74 SW_Push, SW75 SW_Push, SW76 SW_Push, SW77 SW_Push, SW78 SW_Push, SW79 SW_Push, SW8 SW_Push, SW80 SW_Push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

Commit message: Improve routing and board dimensions
Parts:
- moved C2 27.9 mm to (180.1, -33.3), turned to 180 degrees
- moved Y1 27.4 mm to (175.8, -37.5), turned to 315 degrees
- moved C4 24.3 mm to (190.3, -15.2), turned to 0 degrees
- moved C3 20.1 mm to (175.0, -33.3), turned to 0 degrees
- moved D66 1.58 mm to (160.0, -39.8)
- moved C5 0.62 mm to (166.6, -21.8)
Connections:
- net Net-(R1-Pad1) renamed D-
- net Net-(R3-Pad1) renamed D+
Routing:
- net row1: track 589.6 -> 440.3 mm, vias 2 -> 4
- net GND: track 19.9 -> 66.9 mm, vias 209 -> 205
- net Net-(C3-Pad2): track 54.5 -> 8.09 mm, vias 4 -> 0
- net row3: track 501.5 -> 464.4 mm, vias 2 -> 3
- net Net-(C2-Pad2): track 39.9 -> 7.33 mm, vias 2 -> 0
- net D+: track 150.5 -> 126.6 mm, vias 2 -> 0
- net Net-(SW83-Pad2): track 87.1 -> 64.6 mm, vias 1 -> 4
- net col7: track 114.6 -> 136.7 mm, vias 1 -> 2
- net row5: track 461.3 -> 439.2 mm
- net D-: track 146.6 -> 127.3 mm, vias 2 -> 0
- net col9: track 119.4 -> 105.0 mm
- net col3: track 196.9 -> 210.4 mm
- net row4: track 343.2 -> 355.5 mm, vias 4 -> 2
- net col2: track 235.0 -> 246.4 mm
- net col5: track 139.8 -> 150.5 mm, vias 1 -> 3
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Other:
- board size 301 x 111.8 mm -> 298.4 x 109.9 mm

Commit message: Updated footprints
Parts:
- added J2: USB4085-GF-A_REVA, USB4085-GF-A_REVA:GCT_USB4085-GF-A_REVA, F.Cu at (200.7, -132.1)
- D1, D10, D11, D12, D13, D14, D15, D16, D17, D18, D19, D2, D20, D21, D22, D23, D24, D25, D26, D27, D28, D29, D3, D30, D31, D32, D33, D34, D35, D36, D37, D38, D39, D4, D40, D41, D42, D43, D44, D45, D46, D47, D48, D49, D5, D50, D51, D52, D53, D54, D55, D56, D57, D58, D59, D6, D60, D61, D62, D63, D64, D65, D66, D67, D68, D69, D7, D70, D71, D72, D73, D74, D75, D76, D77, D78, D79, D8, D80, D81, D82, D9: footprint Diode_SMD:D_MELF_Handsoldering -> sofaboard:D_SOT-23_ANK
- Y1: value 16MHz -> Crystal_GND24; footprint Cherry:Crytal16 -> Cherry:16MHz Crystal
- moved Y1 3.30 mm to (179.1, -38.1), turned to 0 degrees
Connections:
- Y1 pad 2: Net-(C3-Pad2) -> GND
- Y1 pad 3: (no net) -> Net-(C3-Pad2)

Commit message: reconnect diodes
Parts:
- removed J1: USB_B_Micro, Connector_USB:USB_Micro-B_Amphenol_10103594-0001LF_Horizontal
- moved J2 12.3 mm to (201.0, -119.8), turned to 180 degrees
- moved Y1 4.37 mm to (174.8, -39.0), turned to 225 degrees
- turned D66 to 180 degrees
- turned D67 to 180 degrees
Connections:
- J2 pad A1: Net-(J2-PadA1) -> GND
- J2 pad A12: Net-(J2-PadA1) -> GND
- J2 pad A4: Net-(J2-PadA4) -> +5V
- J2 pad A9: Net-(J2-PadA4) -> +5V
- J2 pad B1: Net-(J2-PadA1) -> GND
- J2 pad B12: Net-(J2-PadA1) -> GND
- J2 pad B4: Net-(J2-PadA4) -> +5V
- J2 pad B6: Net-(J2-PadB6) -> Net-(J2-PadA6)
- J2 pad B7: Net-(J2-PadB7) -> Net-(J2-PadA7)
- J2 pad B9: Net-(J2-PadA4) -> +5V
- J2 pad P1: Net-(J2-PadP1) -> GND
- J2 pad P2: Net-(J2-PadP1) -> GND
- J2 pad P3: Net-(J2-PadP1) -> GND
- J2 pad P4: Net-(J2-PadP1) -> GND
- R1 pad 2: Net-(J1-Pad2) -> Net-(J2-PadA7)
- R3 pad 2: Net-(J1-Pad3) -> Net-(J2-PadA6)
Routing:
- net row1: track 440.3 -> 470.1 mm
- net row3: track 464.4 -> 490.7 mm
- net row5: track 439.2 -> 459.0 mm
- net row4: track 355.5 -> 369.3 mm
- net row0: track 438.0 -> 451.4 mm
- net row2: track 409.9 -> 421.9 mm
- net +5V: track 156.2 -> 163.6 mm
- net GND: track 66.9 -> 60.0 mm, vias 205 -> 226
- net Net-(J2-PadA7): track 0.00 -> 6.09 mm
- net Net-(J2-PadA6): track 0.00 -> 6.01 mm
- net Net-(J1-Pad3): track 5.35 -> 0.00 mm
- net Net-(J1-Pad2): track 5.08 -> 0.00 mm
- net Net-(D65-Pad1): track 13.8 -> 15.6 mm
- net Net-(D67-Pad1): track 7.59 -> 9.45 mm
- net Net-(D75-Pad1): track 10.8 -> 12.5 mm
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
Commit message: refit for order w/einball
Parts:
- added R4: 5.1k, Resistor_SMD:R_0805_2012Metric, B.Cu at (204.5, -109.5)
- added R5: 5.1k, Resistor_SMD:R_0805_2012Metric, B.Cu at (195.5, -109.2)
- added R6: 10k, Resistor_SMD:R_0805_2012Metric, B.Cu at (162.0, -26.8)
- R1, R3: footprint Resistor_SMD:R_0805_2012Metric_Pad1.15x1.40mm_HandSolder -> Resistor_SMD:R_0805_2012Metric
- moved J2 2.75 mm to (201.3, -117.1)
- moved R1 1.27 mm to (200.0, -109.4)
- moved R3 1.27 mm to (202.0, -109.4)
Routing:
- net Net-(J2-PadB5): track 0.00 -> 10.8 mm, vias 0 -> 1
- net +5V: track 163.6 -> 170.7 mm
- net Net-(J2-PadA5): track 0.00 -> 3.49 mm
- net Net-(R6-Pad2): track 64.6 -> 67.8 mm, vias 4 -> 5
- net Net-(J2-PadA6): track 6.01 -> 4.44 mm
- net Net-(J2-PadA7): track 6.09 -> 4.76 mm
- net D-: track 127.3 -> 126.0 mm
- net D+: track 126.6 -> 125.3 mm
- net GND: vias 226 -> 230

Commit message: did more things for final order
Routing:
- net GND: track 60.0 -> 74.5 mm, vias 230 -> 231
